File: pcb/isa-post-card.kicad_pcb (KiCad board)
At the start: 2 copper layers, 107.9 x 64.1 mm, 32 parts, among them J2 POWER, J3 Bus_ISA_8bit_AB_Rev0, J4 Atmel-JTAG-10, SW1 SW_DIP_x05, SW2 SW_DIP_x05, U1 74HCT688, U2 74HCT688, U3 ATF1504AS-xJx44, U5 D168K, U6 D168K

Commit message: Fixing design bugs and adding CUPL code
Parts:
- removed REF**: OSHW-Logo2_7.3x6mm_SilkScreen, Symbol:OSHW-Logo2_7.3x6mm_SilkScreen
- moved RN6 1.80 mm to (67.9, 143.5)
- moved RN5 1.42 mm to (64.1, 143.5)
- moved RN3 1.42 mm to (56.5, 143.5)
- moved RN4 1.27 mm to (60.3, 143.5)
Connections:
- RN3 pad 1: SA0 -> Net-(RN3A-R1.1)
- RN3 pad 2: SA1 -> SA0
- RN3 pad 3: SA2 -> Net-(RN3B-R2.1)
- RN3 pad 4: SA3 -> SA1
- RN3 pad 5: Net-(RN3-R4.2) -> Net-(RN3C-R3.1)
- RN3 pad 6: Net-(RN3-R3.2) -> SA2
- RN3 pad 7: Net-(RN3-R2.2) -> Net-(RN3D-R4.1)
- RN3 pad 8: Net-(RN3-R1.2) -> SA3
- RN4 pad 1: SA4 -> Net-(RN4A-R1.1)
- RN4 pad 2: SA5 -> SA4
- RN4 pad 3: SA6 -> Net-(RN4B-R2.1)
- RN4 pad 4: SA7 -> SA5
- RN4 pad 5: Net-(RN4-R4.2) -> Net-(RN4C-R3.1)
- RN4 pad 6: Net-(RN4-R3.2) -> SA6
- RN4 pad 7: Net-(RN4-R2.2) -> Net-(RN4D-R4.1)
- RN4 pad 8: Net-(RN4-R1.2) -> SA7
- RN5 pad 1: SB0 -> Net-(RN5A-R1.1)
- RN5 pad 2: SB1 -> SB0
- RN5 pad 3: SB2 -> Net-(RN5B-R2.1)
- RN5 pad 4: SB3 -> SB1
- RN5 pad 5: Net-(RN5-R4.2) -> Net-(RN5C-R3.1)
- RN5 pad 6: Net-(RN5-R3.2) -> SB2
- RN5 pad 7: Net-(RN5-R2.2) -> Net-(RN5D-R4.1)
- RN5 pad 8: Net-(RN5-R1.2) -> SB3
- RN6 pad 1: SB4 -> Net-(RN6A-R1.1)
- RN6 pad 2: SB5 -> SB4
- RN6 pad 3: SB6 -> Net-(RN6B-R2.1)
- RN6 pad 4: SB7 -> SB5
- RN6 pad 5: Net-(RN6-R4.2) -> Net-(RN6C-R3.1)
- RN6 pad 6: Net-(RN6-R3.2) -> SB6
- RN6 pad 7: Net-(RN6-R2.2) -> Net-(RN6D-R4.1)
- RN6 pad 8: Net-(RN6-R1.2) -> SB7
- U5 pad 1: Net-(RN4-R1.2) -> Net-(RN4A-R1.1)
- U5 pad 10: Net-(RN4-R3.2) -> Net-(RN4C-R3.1)
- U5 pad 2: Net-(RN3-R4.2) -> Net-(RN3D-R4.1)
- U5 pad 4: Net-(RN3-R3.2) -> Net-(RN3C-R3.1)
- U5 pad 5: Net-(RN4-R4.2) -> Net-(RN4D-R4.1)
- U5 pad 6: Net-(RN3-R2.2) -> Net-(RN3B-R2.1)
- U5 pad 7: Net-(RN3-R1.2) -> Net-(RN3A-R1.1)
- U5 pad 9: Net-(RN4-R2.2) -> Net-(RN4B-R2.1)
- U6 pad 1: Net-(RN6-R1.2) -> Net-(RN6A-R1.1)
- U6 pad 10: Net-(RN6-R3.2) -> Net-(RN6C-R3.1)
- U6 pad 2: Net-(RN5-R4.2) -> Net-(RN5D-R4.1)
- U6 pad 4: Net-(RN5-R3.2) -> Net-(RN5C-R3.1)
- U6 pad 5: Net-(RN6-R4.2) -> Net-(RN6D-R4.1)
- U6 pad 6: Net-(RN5-R2.2) -> Net-(RN5B-R2.1)
- U6 pad 7: Net-(RN5-R1.2) -> Net-(RN5A-R1.1)
- U6 pad 9: Net-(RN6-R2.2) -> Net-(RN6B-R2.1)
Routing:
- net SA0: track 66.8 -> 0.00 mm, vias 2 -> 0
- net Net-(RN4-R1.2): track 40.5 -> 0.00 mm, vias 1 -> 0
- net SA5: track 38.7 -> 0.00 mm
- net SB6: track 37.2 -> 0.00 mm
- net Net-(RN6-R1.2): track 37.1 -> 0.00 mm, vias 2 -> 0
- net Net-(RN4-R3.2): track 34.6 -> 0.00 mm
- net SB3: track 33.9 -> 0.00 mm
- net Net-(RN3-R4.2): track 33.1 -> 0.00 mm
- net SA2: track 32.4 -> 0.00 mm
- net Net-(RN4-R2.2): track 32.1 -> 0.00 mm
- net Net-(RN6-R3.2): track 32.0 -> 0.00 mm
- net SA1: track 31.7 -> 0.00 mm
- net SB5: track 31.2 -> 0.00 mm
- net SB7: track 29.7 -> 0.00 mm
- net Net-(RN6-R2.2): track 29.6 -> 0.00 mm, vias 1 -> 0
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Other:
- board text removed: "ISA POST CARD"

Commit message: Fixing board wiring
Routing:
- net Net-(RN4B-R2.1): track 0.00 -> 51.2 mm
- net Net-(RN5C-R3.1): track 0.00 -> 48.7 mm, vias 0 -> 1
- net SB6: track 0.00 -> 44.5 mm, vias 0 -> 1
- net Net-(RN4C-R3.1): track 0.00 -> 43.1 mm, vias 0 -> 1
- net SA0: track 0.00 -> 43.0 mm, vias 0 -> 1
- net Net-(RN3D-R4.1): track 0.00 -> 42.6 mm
- net Net-(RN5D-R4.1): track 0.00 -> 40.3 mm, vias 0 -> 1
- net SB7: track 0.00 -> 39.7 mm, vias 0 -> 2
- net Net-(RN6B-R2.1): track 0.00 -> 38.9 mm
- net SB3: track 0.00 -> 38.8 mm, vias 0 -> 1
- net SA6: track 0.00 -> 36.8 mm, vias 0 -> 1
- net Net-(RN4A-R1.1): track 0.00 -> 35.5 mm
- net SA2: track 0.00 -> 32.1 mm
- net Net-(RN4D-R4.1): track 0.00 -> 31.5 mm, vias 0 -> 1
- net SA3: track 0.00 -> 31.4 mm, vias 0 -> 1
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
Commit message: Revising design
Parts:
- added REF**: OSHW-Logo2_14.6x12mm_SilkScreen, Symbol:OSHW-Logo2_14.6x12mm_SilkScreen, F.Cu at (110.5, 160.0)
- moved C1 96.9 mm to (116.6, 115.6)
- moved J4 60.3 mm to (83.8, 104.1)
- moved C6 59.1 mm to (39.4, 163.9)
- moved RN2 43.8 mm to (99.1, 158.8)
- moved J2 36.0 mm to (71.1, 115.6)
- moved C7 29.6 mm to (91.4, 152.4), turned to 180 degrees
- moved U2 26.7 mm to (76.2, 170.2)
- moved U1 25.4 mm to (43.2, 170.2)
- moved U5 25.0 mm to (37.5, 118.0)
- moved U6 25.0 mm to (50.8, 118.0)
- moved D2 23.6 mm to (101.6, 104.1)
- moved D3 23.6 mm to (108.6, 104.1)
- moved D4 23.6 mm to (115.6, 104.1)
- moved R1 23.6 mm to (101.6, 119.4)
- moved R4 23.6 mm to (111.1, 119.4)
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Routing:
- net GND: track 631.0 -> 214.1 mm, vias 0 -> 3
- net +5V: track 424.3 -> 293.8 mm, vias 1 -> 8
- net Net-(RN1-R4): track 75.5 -> 16.1 mm
- net Net-(RN2-R5): track 119.6 -> 68.8 mm
- net Net-(RN2-R4): track 113.2 -> 64.3 mm
- net A0: track 61.1 -> 16.9 mm
- net Net-(RN2-R8): track 88.7 -> 46.3 mm
- net Net-(RN2-R7): track 93.7 -> 52.4 mm
- net Net-(RN2-R6): track 108.6 -> 67.4 mm, vias 0 -> 1
- net ~{SEL1}: track 27.2 -> 62.4 mm
- net A5: track 68.8 -> 34.6 mm, vias 0 -> 1
- net Net-(RN1-R6): track 60.1 -> 26.2 mm
- net Net-(RN1-R5): track 61.5 -> 28.5 mm
- net AEN: track 45.5 -> 76.8 mm, vias 2 -> 4
- net A4: track 60.6 -> 30.1 mm, vias 1 -> 0
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- added copper zone on B.Cu, net +5V
- added copper zone on F.Cu, net GND
- removed copper zone on F.Cu, net +5V
- removed copper zone on B.Cu, net GND
Other:
- board size 107.9 x 64.1 mm -> 87.5 x 86.4 mm
- board text added: "ISA POST CARD rev1"
- board text added: "jlcjlcjlcjlc"

Commit message: Revising schematics
Parts:
- removed REF**: OSHW-Logo2_14.6x12mm_SilkScreen, Symbol:OSHW-Logo2_14.6x12mm_SilkScreen
- added C8: 100n, Capacitor_THT:C_Disc_D5.0mm_W2.5mm_P5.00mm, F.Cu at (113.0, 149.2)
- added D5: CLK, LED_THT:LED_D5.0mm, F.Cu at (94.0, 114.3)
- added D6: RESET, LED_THT:LED_D5.0mm, F.Cu at (101.6, 114.3)
- added R5: 1k, Resistor_THT:R_Axial_DIN0207_L6.3mm_D2.5mm_P7.62mm_Horizontal, F.Cu at (114.9, 129.5)
- added R6: 500, Resistor_THT:R_Axial_DIN0207_L6.3mm_D2.5mm_P7.62mm_Horizontal, F.Cu at (118.1, 129.5)
- added U4: 74HC00, Package_DIP:DIP-14_W7.62mm_Socket, F.Cu at (106.7, 154.3)
- J4: value Atmel-JTAG-10 -> PROGRAMMER
- moved J4 43.1 mm to (52.7, 134.0)
- moved C1 30.8 mm to (86.4, 109.9)
- moved RN5 21.6 mm to (66.0, 120.7), turned to 90 degrees
- moved RN6 20.7 mm to (69.8, 120.7), turned to 90 degrees
- moved RN3 18.9 mm to (38.1, 123.2), turned to 0 degrees
- moved RN4 17.8 mm to (38.1, 126.4), turned to 0 degrees
- moved J2 11.0 mm to (79.6, 108.6)
- moved R1 10.2 mm to (102.2, 129.5)
- moved R2 10.2 mm to (105.4, 129.5)
- moved R3 10.2 mm to (108.6, 129.5)
- moved R4 10.2 mm to (111.8, 129.5)
- moved C3 5.00 mm to (72.4, 163.9), turned to -90 degrees
- moved U3 2.84 mm to (87.6, 132.1)
- moved C2 2.84 mm to (83.9, 121.9)
- moved C7 2.84 mm to (88.8, 153.7)
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Connections:
- J3 pad B20: unconnected-(J3-CLK-PadB20) -> CLK
- RN3 pad 2: SA0 -> SA4
- RN3 pad 4: SA1 -> SA3
- RN3 pad 8: SA3 -> SA7
- RN4 pad 2: SA4 -> SA6
- RN4 pad 6: SA6 -> SA0
- RN4 pad 8: SA7 -> SA1
- RN5 pad 2: SB0 -> SB2
- RN5 pad 4: SB1 -> SB7
- RN5 pad 6: SB2 -> SB1
- RN5 pad 8: SB3 -> SB0
- RN6 pad 4: SB5 -> SB3
- RN6 pad 6: SB6 -> SB5
- RN6 pad 8: SB7 -> SB6
- U3 pad 11: unconnected-(U3-I/O/PD1-Pad11) -> SA2
- U3 pad 12: SA5 -> SA1
- U3 pad 14: SA6 -> SA0
- U3 pad 16: SA7 -> SA3
- U3 pad 17: SB0 -> SA5
- U3 pad 18: SB1 -> SA6
- U3 pad 19: SB2 -> SA4
- U3 pad 20: SB3 -> D0
- U3 pad 21: SB4 -> D1
- U3 pad 24: SB5 -> D2
- U3 pad 25: unconnected-(U3-I/O/PD2-Pad25) -> D3
- U3 pad 26: SB6 -> D4
- U3 pad 27: SB7 -> D5
- U3 pad 28: ~{SEL1} -> D6
- U3 pad 29: D0 -> D7
- U3 pad 31: D1 -> ~{SEL2}
- U3 pad 33: D2 -> unconnected-(U3-I/O-Pad33)
- U3 pad 34: D3 -> ~{SEL1}
- U3 pad 36: D4 -> unconnected-(U3-I/O-Pad36)
- U3 pad 37: D5 -> SB0
- U3 pad 39: D6 -> SB6
- U3 pad 4: SA0 -> SB4
- U3 pad 40: D7 -> SB1
- U3 pad 41: ~{SEL2} -> SB5
- U3 pad 5: SA1 -> SB3
- U3 pad 6: SA2 -> SB2
- U3 pad 8: SA3 -> SB7
- U3 pad 9: SA4 -> SA7
- U5 pad 1: Net-(RN4A-R1.1) -> Net-(RN3A-R1.1)
- U5 pad 10: Net-(RN4C-R3.1) -> Net-(RN4A-R1.1)
- U5 pad 2: Net-(RN3D-R4.1) -> Net-(RN3B-R2.1)
- U5 pad 5: Net-(RN4D-R4.1) -> Net-(RN3D-R4.1)
- U5 pad 6: Net-(RN3B-R2.1) -> Net-(RN4D-R4.1)
- U5 pad 7: Net-(RN3A-R1.1) -> Net-(RN4C-R3.1)
- U6 pad 10: Net-(RN6C-R3.1) -> Net-(RN6D-R4.1)
- U6 pad 2: Net-(RN5D-R4.1) -> Net-(RN6B-R2.1)
- U6 pad 4: Net-(RN5C-R3.1) -> Net-(RN5A-R1.1)
- U6 pad 5: Net-(RN6D-R4.1) -> Net-(RN5B-R2.1)
- U6 pad 6: Net-(RN5B-R2.1) -> Net-(RN5C-R3.1)
- U6 pad 7: Net-(RN5A-R1.1) -> Net-(RN5D-R4.1)
- U6 pad 9: Net-(RN6B-R2.1) -> Net-(RN6C-R3.1)
Routing:
- net GND: track 214.1 -> 635.2 mm, vias 3 -> 9
- net +5V: track 293.8 -> 428.8 mm, vias 8 -> 1
- net CLK: track 0.00 -> 61.5 mm, vias 0 -> 2
- net Net-(R6-Pad1): track 0.00 -> 45.7 mm, vias 0 -> 2
- net Net-(RN5B-R2.1): track 42.6 -> 6.08 mm
- net Net-(RN5A-R1.1): track 45.0 -> 8.72 mm
- net Net-(R5-Pad1): track 0.00 -> 34.2 mm
- net Net-(RN3A-R1.1): track 37.6 -> 5.47 mm
- net SB7: track 58.9 -> 28.2 mm, vias 0 -> 1
- net Net-(D5-A): track 0.00 -> 26.6 mm, vias 0 -> 1
- net SB0: track 28.2 -> 53.9 mm, vias 0 -> 1
- net Net-(RN3B-R2.1): track 33.2 -> 7.63 mm
- net Net-(RN6C-R3.1): track 48.1 -> 24.6 mm
- net Net-(RN6B-R2.1): track 41.9 -> 18.5 mm
- net SA7: track 51.1 -> 28.9 mm
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Other:
- board text added: "ISA POST CARD"
- board text added: "THIS SIDE IS FACING BACK"
- board text removed: "+"
- board text removed: "-"
- board text removed: "ISA POST CARD rev1"
